File: hdw/drewSBC/DDR3.kicad_sch (KiCad schematic)
At the start: 0 parts

Commit message: added DDR3 sheet
Parts:
- added C? (x17): 0.1uF, Capacitors_SMD:C_0402, symbol Custom_Library:C_Custom
- added C?: 1nF, Capacitors_SMD:C_0402, symbol Custom_Library:C_Custom
- added R?: 1.5k, Resistors_SMD:R_0402, symbol Custom_Library:R_Custom
- added R? (x3): 10k, Resistors_SMD:R_0402, symbol Custom_Library:R_Custom
- added R?: 240, Resistors_SMD:R_0402, symbol Custom_Library:R_Custom
- added U?: AS4C256M16D3, Package_BGA:BGA-96_9.0x13.0mm_Layout2x3x16_P0.8mm, symbol Memory_RAM:AS4C256M16D3
Connections:
- new net: R?.1, U?.L8 (ZQ)
- new net DDR_A0: U?.N3 (A0)
- new net DDR_A1: U?.P7 (A1)
- new net DDR_A10: U?.L7 (A10/AP)
- new net DDR_A11: U?.R7 (A11)
- new net DDR_A12: U?.N7 (A12/~{BC})
- new net DDR_A13: U?.T3 (A13)
- new net DDR_A14: U?.T7 (A14)
- new net DDR_A2: U?.P3 (A2)
- new net DDR_A3: U?.N2 (A3)
- new net DDR_A4: U?.P8 (A4)
- new net DDR_A5: U?.P2 (A5)
- new net DDR_A6: U?.R8 (A6)
- new net DDR_A7: U?.R2 (A7)
- new net DDR_A8: U?.T8 (A8)
- new net DDR_A9: U?.R3 (A9)
- new net DDR_BA0: U?.M2 (BA0)
- new net DDR_BA1: U?.N8 (BA1)
- new net DDR_BA2: U?.M3 (BA2)
- new net DDR_CK: U?.J7 (CK)
- new net DDR_CKE: R?.1, U?.K9 (CKE)
- new net DDR_DQ0: U?.E3 (DQ0)
- new net DDR_DQ1: U?.F7 (DQ1)
- new net DDR_DQ10: U?.C8 (DQ10)
- new net DDR_DQ11: U?.C2 (DQ11)
- new net DDR_DQ12: U?.A7 (DQ12)
- new net DDR_DQ13: U?.A2 (DQ13)
- new net DDR_DQ14: U?.B8 (DQ14)
- new net DDR_DQ15: U?.A3 (DQ15)
- new net DDR_DQ2: U?.F2 (DQ2)
- new net DDR_DQ3: U?.F8 (DQ3)
- new net DDR_DQ4: U?.H3 (DQ4)
- new net DDR_DQ5: U?.H8 (DQ5)
- new net DDR_DQ6: U?.G2 (DQ6)
- new net DDR_DQ7: U?.H7 (DQ7)
- new net DDR_DQ8: U?.D7 (DQ8)
- new net DDR_DQ9: U?.C3 (DQ9)
- new net DDR_DQM0: U?.E7 (LDM)
- new net DDR_DQM1: U?.D3 (UDM)
- new net DDR_DQS0: U?.F3 (LDQS)
- new net DDR_DQS1: U?.C7 (UDQS)
- new net DDR_ODT: U?.K1 (ODT)
- new net DDR_VREF: C?.1, C?.1, R?.1, R?.2, U?.H1 (VREFDQ), U?.M8 (VREFCA)
- new net GND: C?.2, C?.2, C?.2, C?.2, C?.2, C?.2, C?.2, C?.2, C?.2, C?.2, C?.2, C?.2, C?.2, C?.2, C?.2, C?.2, C?.2, C?.2, R?.2, R?.2, R?.2, U?.A9 (VSS), U?.B1 (VSSQ), U?.B3 (VSS), U?.B9 (VSSQ), U?.D1 (VSSQ), U?.D8 (VSSQ), U?.E1 (VSS), U?.E2 (VSSQ), U?.E8 (VSSQ), U?.F9 (VSSQ), U?.G1 (VSSQ), U?.G8 (VSS), U?.G9 (VSSQ), U?.J2 (VSS), U?.J8 (VSS), U?.M1 (VSS), U?.M9 (VSS), U?.P1 (VSS), U?.P9 (VSS), U?.T1 (VSS), U?.T9 (VSS)
- new net VMEM: C?.1, C?.1, C?.1, C?.1, C?.1, C?.1, C?.1, C?.1, C?.1, C?.1, C?.1, C?.1, C?.1, C?.1, C?.1, C?.1, R?.1, R?.1, U?.A1 (VDDQ), U?.A8 (VDDQ), U?.B2 (VDD), U?.C1 (VDDQ), U?.C9 (VDDQ), U?.D2 (VDDQ), U?.D9 (VDD), U?.E9 (VDDQ), U?.F1 (VDDQ), U?.G7 (VDD), U?.H2 (VDDQ), U?.H9 (VDDQ), U?.K2 (VDD), U?.K8 (VDD), U?.N1 (VDD), U?.N9 (VDD), U?.R1 (VDD), U?.R9 (VDD)
- new net ~{DDR_CAS}: U?.K3 (~{CAS})
- new net ~{DDR_CK}: U?.K7 (~{CK})
- new net ~{DDR_CS}: U?.L2 (~{CS})
- new net ~{DDR_DQS0}: U?.G3 (~{LDQS})
- new net ~{DDR_DQS1}: U?.B7 (~{UDQS})
- new net ~{DDR_RAS}: U?.J3 (~{RAS})
- new net ~{DDR_RESET}: R?.2, U?.T2 (~{RESET})
- new net ~{DDR_WE}: U?.L3 (~{WE})
