File: hdw/drewSBC/Sitara6.kicad_sch (KiCad schematic)
At the start: 0 parts

Commit message: ripped up ETH phy
Parts:
- added R? (x32): 100k, Resistors_SMD:R_0402, symbol Custom_Library:R_Custom
Connections:
- new net +3.3V: R?.2, R?.2, R?.2, R?.2, R?.2, R?.2, R?.2, R?.2, R?.2, R?.2, R?.2, R?.2, R?.2, R?.2, R?.2, R?.2
- new net GND: R?.1, R?.1, R?.1, R?.1, R?.1, R?.1, R?.1, R?.1, R?.1, R?.1, R?.1, R?.1, R?.1, R?.1, R?.1, R?.1
- new net LCD_DATA0: R?.1, R?.2
- new net LCD_DATA1: R?.1, R?.2
- new net LCD_DATA10: R?.1, R?.2
- new net LCD_DATA11: R?.1, R?.2
- new net LCD_DATA12: R?.1, R?.2
- new net LCD_DATA13: R?.1, R?.2
- new net LCD_DATA14: R?.1, R?.2
- new net LCD_DATA15: R?.1, R?.2
- new net LCD_DATA2: R?.1, R?.2
- new net LCD_DATA3: R?.1, R?.2
- new net LCD_DATA4: R?.1, R?.2
- new net LCD_DATA5: R?.1, R?.2
- new net LCD_DATA6: R?.1, R?.2
- new net LCD_DATA7: R?.1, R?.2
- new net LCD_DATA8: R?.1, R?.2
- new net LCD_DATA9: R?.1, R?.2
